Commit message: feat: add LIDAR link and joints to URDF, update monitoring scripts for improved functionality

File: core_ws/src/bungy_description/urdf/bungy_robot.urdf.xacro (robot description, xacro)
@@ -27,5 +27,5 @@
     </inertial>
   </link>
-  <!-- Left wheel link -->
+    <!-- Left wheel link -->
   <link name="left_wheel_link">
     <visual>
@@ -81,4 +81,64 @@
     <axis xyz="0 0 1"/>
   </joint>
+  <!-- LIDAR Link -->
+  <link name="laser_link">
+    <visual>
+      <geometry>
+        <cylinder radius="0.05" length="0.04"/>
+      </geometry>
+      <material name="red">
+        <color rgba="1.0 0.0 0.0 1.0"/>
+      </material>
+    </visual>
+    <collision>
+      <geometry>
+        <cylinder radius="0.05" length="0.04"/>
+      </geometry>
+    </collision>
+    <inertial>
+      <mass value="0.125"/>
+      <inertia ixx="0.001" ixy="0.0" ixz="0.0" iyy="0.001" iyz="0.0" izz="0.001"/>
+    </inertial>
+  </link>
+  <!-- LIDAR Joint -->
+  <joint name="laser_joint" type="fixed">
+    <parent link="base_link"/>
+    <child link="laser_link"/>
+    <origin xyz="0.08 0.0 0.09" rpy="0 0 0"/>
+  </joint>
+  <!-- Right wheel link -->
+  <link name="right_wheel_joint">
+    <visual>
+      <geometry>
+        <cylinder radius="${wheel_radius}" length="0.05"/>
+      </geometry>
+      <material name="black">
+        <color rgba="0.0 0.0 0.0 1.0"/>
+      </material>
+    </visual>
+    <collision>
+      <geometry>
+        <cylinder radius="${wheel_radius}" length="0.05"/>
+      </geometry>
+    </collision>
+    <inertial>
+      <mass value="0.1"/>
+      <inertia ixx="0.001" ixy="0.0" ixz="0.0" iyy="0.001" iyz="0.0" izz="0.001"/>
+    </inertial>
+  </link>
+  <!-- Left wheel joint -->
+  <joint name="left_wheel_joint_connector" type="continuous">
+    <parent link="base_link"/>
+    <child link="left_wheel_joint"/>
+    <origin xyz="0.0 ${wheel_separation/2} 0.0" rpy="-${pi/2} 0 0"/>
+    <axis xyz="0 0 1"/>
+  </joint>
+  <!-- Right wheel joint -->
+  <joint name="right_wheel_joint_connector" type="continuous">
+    <parent link="base_link"/>
+    <child link="right_wheel_joint"/>
+    <origin xyz="0.0 -${wheel_separation/2} 0.0" rpy="-${pi/2} 0 0"/>
+    <axis xyz="0 0 1"/>
+  </joint>
   <!-- Conditional ros2_control inclusion -->
   <xacro:if value="$(arg use_ros2_control)">

Commit message: feat: refactor URDF and launch files for improved robot configuration and control

File: core_ws/src/bungy_description/urdf/bungy_robot.urdf.xacro (robot description, xacro)
@@ -107,38 +107,4 @@
     <origin xyz="0.08 0.0 0.09" rpy="0 0 0"/>
   </joint>
-  <!-- Right wheel link -->
-  <link name="right_wheel_joint">
-    <visual>
-      <geometry>
-        <cylinder radius="${wheel_radius}" length="0.05"/>
-      </geometry>
-      <material name="black">
-        <color rgba="0.0 0.0 0.0 1.0"/>
-      </material>
-    </visual>
-    <collision>
-      <geometry>
-        <cylinder radius="${wheel_radius}" length="0.05"/>
-      </geometry>
-    </collision>
-    <inertial>
-      <mass value="0.1"/>
-      <inertia ixx="0.001" ixy="0.0" ixz="0.0" iyy="0.001" iyz="0.0" izz="0.001"/>
-    </inertial>
-  </link>
-  <!-- Left wheel joint -->
-  <joint name="left_wheel_joint_connector" type="continuous">
-    <parent link="base_link"/>
-    <child link="left_wheel_joint"/>
-    <origin xyz="0.0 ${wheel_separation/2} 0.0" rpy="-${pi/2} 0 0"/>
-    <axis xyz="0 0 1"/>
-  </joint>
-  <!-- Right wheel joint -->
-  <joint name="right_wheel_joint_connector" type="continuous">
-    <parent link="base_link"/>
-    <child link="right_wheel_joint"/>
-    <origin xyz="0.0 -${wheel_separation/2} 0.0" rpy="-${pi/2} 0 0"/>
-    <axis xyz="0 0 1"/>
-  </joint>
   <!-- Conditional ros2_control inclusion -->
   <xacro:if value="$(arg use_ros2_control)">
