Commit message: feat: restructure URDF files and launch configurations for improved robot representation and control

File: monitoring_ws/src/bungy_monitoring/urdf/bungy_visual.urdf.xacro (robot description, xacro)
@@ -1,23 +1,31 @@
 <?xml version="1.0"?>
-<robot xmlns:xacro="http://www.ros.org/wiki/xacro" name="bungy">
-  <!-- Parameters -->
-  <xacro:arg name="use_ros2_control" default="false" />
-  <xacro:arg name="use_sim_time" default="false" />
-  <!-- Robot physical properties -->
+<robot xmlns:xacro="http://www.ros.org/wiki/xacro" name="bungy_visual">
+  <!-- Robot physical properties - need to redeclare for access -->
   <xacro:property name="wheel_separation" value="0.184" />
   <xacro:property name="wheel_radius" value="0.06" />
-  <!-- Base link -->
+  <xacro:property name="base_width" value="0.25" />
+  <xacro:property name="base_length" value="0.15" />
+  <xacro:property name="base_height" value="0.1" />
+  <!-- Materials for visualization -->
+  <material name="blue">
+    <color rgba="0.0 0.0 1.0 1.0"/>
+  </material>
+  <material name="black">
+    <color rgba="0.0 0.0 0.0 1.0"/>
+  </material>
+  <material name="red">
+    <color rgba="1.0 0.0 0.0 1.0"/>
+  </material>
+  <!-- Base link with visuals -->
   <link name="base_link">
     <visual>
       <geometry>
-        <box size="0.25 0.15 0.1"/>
+        <box size="${base_width} ${base_length} ${base_height}"/>
       </geometry>
-      <material name="blue">
-        <color rgba="0.0 0.0 1.0 1.0"/>
-      </material>
+      <material name="blue"/>
     </visual>
     <collision>
       <geometry>
-        <box size="0.25 0.15 0.1"/>
+        <box size="${base_width} ${base_length} ${base_height}"/>
       </geometry>
     </collision>
@@ -27,5 +35,5 @@
     </inertial>
   </link>
-    <!-- Left wheel link -->
+  <!-- Left wheel link with visuals -->
   <link name="left_wheel_link">
     <visual>
@@ -33,7 +41,5 @@
         <cylinder radius="${wheel_radius}" length="0.05"/>
       </geometry>
-      <material name="black">
-        <color rgba="0.0 0.0 0.0 1.0"/>
-      </material>
+      <material name="black"/>
     </visual>
     <collision>
@@ -47,5 +53,5 @@
     </inertial>
   </link>
-  <!-- Right wheel link -->
+  <!-- Right wheel link with visuals -->
   <link name="right_wheel_link">
     <visual>
@@ -53,7 +59,5 @@
         <cylinder radius="${wheel_radius}" length="0.05"/>
       </geometry>
-      <material name="black">
-        <color rgba="0.0 0.0 0.0 1.0"/>
-      </material>
+      <material name="black"/>
     </visual>
     <collision>
@@ -81,5 +85,5 @@
     <axis xyz="0 0 1"/>
   </joint>
-  <!-- LIDAR Link -->
+  <!-- LIDAR link with visuals -->
   <link name="laser_link">
     <visual>
@@ -87,7 +91,5 @@
         <cylinder radius="0.05" length="0.04"/>
       </geometry>
-      <material name="red">
-        <color rgba="1.0 0.0 0.0 1.0"/>
-      </material>
+      <material name="red"/>
     </visual>
     <collision>
@@ -101,5 +103,5 @@
     </inertial>
   </link>
-  <!-- LIDAR Joint -->
+  <!-- LIDAR joint -->
   <joint name="laser_joint" type="fixed">
     <parent link="base_link"/>
@@ -107,7 +109,3 @@
     <origin xyz="0.08 0.0 0.09" rpy="0 0 0"/>
   </joint>
-  <!-- Conditional ros2_control inclusion -->
-  <xacro:if value="$(arg use_ros2_control)">
-    <xacro:include filename="$(find bungy_description)/urdf/bungy_robot.ros2_control.xacro" />
-  </xacro:if>
 </robot>
